File: Adafruit_TMP117.sch (EAGLE design)
At the start: 16 parts, among them X1 TMP117_WSON

Commit message: changed in to a smaller layout with a "finger" and single connector
Parts:
- removed CONN3: STEMMA_I2C_QT, microbuilder:STEMMA_I2C_QT
- removed D1: GREEN, microbuilder:LED0603_NOOUTLINE
- removed FID3, FID4: FIDUCIAL_1MM, microbuilder:FIDUCIAL_1MM
- removed JP1: (no value), microbuilder:HEADER-1X670MIL
- removed SJ1: (no value), microbuilder:SOLDERJUMPER
- removed U$17, U$21: MOUNTINGHOLE2.5, microbuilder:MOUNTINGHOLE2.5
- added R2, R4: 10k, rcl:R-EU_R0402
- added R6: 0R, rcl:R-EU_R0402
- C1: device microbuilder:CAP_CERAMIC0603_NO -> microbuilder:CAP_CERAMIC_0402
- C2: device microbuilder:CAP_CERAMIC0805-NOOUTLINE -> microbuilder:CAP_CERAMIC_0603
- R1: value (none) -> 10k; device microbuilder:RESISTOR_0603_NOOUT -> rcl:R-EU_R0402
- R3: value 10K -> 10k; device microbuilder:RESISTOR_4PACK -> rcl:R-EU_R0402
Connections:
- removed net N$1: D1.A, R1.1
- net ADDR: now also R2.1, R6.1; no longer JP1.6, R3G$1.2, SJ1.1
- net GND: now also R2.2; no longer CONN3G$1.GND, CONN3G$2.MT, CONN3G$3.MT, D1.C, JP1.2, R3G$1.1
- net INT: now also R1.1; no longer JP1.5, R3G$2.2
- net SCL: now also R3.1; no longer CONN3G$1.SCL, JP1.3, R3G$4.1
- net SDA: now also R4.1; no longer CONN3G$1.SDA, JP1.4, R3G$3.1
- net VCC: now also R3.2, R4.2, R6.2; no longer CONN3G$1.V+, JP1.1, R3G$2.1, R3G$3.2, R3G$4.2, SJ1.2
Other:
- note removed: "ON LED"
- moved on the sheet: R1, R3

Commit message: new version, sensors on bottom side, connector on top side. Two sensors with I2C in series.
Parts:
- removed R1, R2: 10k, rcl:R-EU_R0402
- removed R6: 0R, rcl:R-EU_R0402
- added C3: 0.1uF, microbuilder:CAP_CERAMIC_0402
- added X2: TMP117_WSON, adafruit_sensor:TMP117_WSON
Connections:
- removed net ADDR: R2.1, R6.1, X1.ADDR
- removed net INT: R1.1, X1.ALERT
- net GND: now also C3.2, X1.ALERT, X2.ADDR, X2.ALERT, X2.VSS; no longer R2.2
- net SCL: now also X2.SCL
- net SDA: now also X2.SDA
- net VCC: now also C3.1, X1.ADDR, X2.VDD; no longer R1.2, R6.2
